File: monKWH+GPS/untitled.sch (EAGLE design)
At the start: 61 parts, among them J1 U.FL-R-SMT(01), J3 2172034-1, J4 POWER_JACKSLT, Q1 MMBT3904, Q2 MMBT3904, Q3 12MHz, Q4 MC-306, U2 DS1307Z+, U3 MAX3444EASA, U4 AMS1117, U5 MAX232CSE, X1 MSTBA2

Commit message: revisi rangkaian
Parts:
- removed C13, C15, C16, C17, C18: 10uf/50V, EEEFK1H100V:EEEFK1H100V
- removed D2: Tx, LHN974_RED_LED_1206:LHN974_RED_LED_1206
- removed D3: Rx, LHN974_RED_LED_1206:LHN974_RED_LED_1206
- removed G1: CR2032H, battery_cr2032:CR2032H
- removed J2: (no value), SparkFun-Connectors:DB9FEMALE
- removed Q4: MC-306, crystal:MC-306
- removed R10, R6, R9: 10K, adafruit:R-US_M0805
- removed U$1: STEPDOWN_SY8205, STEPDOWN_SY8205:STEPDOWN_SY8205
- added C19, C20, C21, C5, C9: 10uF, rcl:C-EUC0805K
- added C25: 10uF/16v, rcl:CPOL-EU153CLV-0505
- added C26, C28, C30, C31, C32: 10uF/16V, rcl:CPOL-EU153CLV-0505
- added C27: 0.1uF/16V, rcl:CPOL-EU153CLV-0505
- added C29: 0.1uf/16V, rcl:CPOL-EU153CLV-0505
- added J5: RJ45-8N-B, RJ45-8N-B:RJ45-8N-B
- added U1: RT9193-33GB, RT9193-33GB:RT9193-33GB
- C11: value 10uf/50V -> 10uF; device EEEFK1H100V:EEEFK1H100V -> rcl:C-EUC0805K
- C4: value 10uf/50V -> 10uF/16V; device EEEFK1H100V:EEEFK1H100V -> rcl:CPOL-EU153CLV-0505
- D1, D6: value 1N5819HW-7 -> SML-LXT0805IW-TR; device 1N5819HW-7:1N5819HW-7 -> SML-LXT0805IW-TR:SML-LXT0805IW-TR
- U2: value DS1307Z+ -> RT9193-33GB; device DS1307Z_:DS1307Z+ -> RT9193-33GB:RT9193-33GB
- U3: value MAX3444EASA -> RT9193-33GB; device MAX3444EASA:MAX3444EASA -> RT9193-33GB:RT9193-33GB
- U4: value AMS1117 -> L80-R; device AMS1117:AMS1117 -> L80-R:L80-R
Connections:
- removed net CLK: MD1.CLK
- removed net CMD: MD1.CMD
- removed net IO34: MD1.IO34
- removed net IO35: MD1.IO35
- removed net N$11: D4.A, U$1.OUT_VCC
- removed net N$15: G1.+, U2.VBAT
- removed net N$18: R10.1, U2.SQW/OUT
- removed net N$20: D1.A, J2.9
- removed net N$23: D6.A, J4.PWR
- removed net N$7: Q4.2, U2.X2
- removed net NC: MD1.NC
- removed net RST_LAN: MD1.IO21, U$3.RST
- removed net SCL: R9.2, U2.SCL, U3.A
- removed net SD0: MD1.SD0
- removed net SD1: MD1.SD1
- removed net SD2: MD1.SD2
- removed net SD3: MD1.SD3
- removed net SDA: R6.2, U2.SDA, U3.GND
- removed net SENSOR_VN: MD1.SENSOR_VN
- removed net SENSOR_VP: MD1.SENSOR_VP
- removed net VCC_DB9: D6.K, U$1.IN_VCC
- new net 3V3-LAN-GPS: C21.1, C27.+, C28.+, C29.+, U$3.3V3, U$3.3V3.2, U3.VOUT, U4.VCC, U4.V_BCKP
- new net 3V3-LORA-RS232: C19.1, C4.-, C7.2, C8.2, LORA-NICERF-V1.VCC, U2.VOUT, U5.VCC
- new net EN-3V3-LAN-GPS: MD1.IO33, U3.EN
- new net GPS_RXD: MD1.IO22, U4.RXD1
- new net GPS_TXD: MD1.IO21, U4.TXD1
- net 3V3: now also C9.1, U1.VOUT; no longer C11.1, C16.2, C7.2, C8.2, LORA-NICERF-V1.VCC, U4.VOUT, U5.VCC
- net GND: now also C19.2, C20.2, C21.2, C25.-, C26.-, C27.-, C28.-, C29.-, C32.+, C5.2, C9.2, J5.6, J5.SHIELD, U1.GND, U3.GND, U4.GND; no longer C17.1, C18.2, C4.2, G1.-, J2.5, U$1.IN_GND, U$1.OUT_GND, U3.!DE, U3.!RE, U3.B, U3.RO, U3.TXD, U4.ADJ/GND
- net INT_LAN: no longer MD1.IO22
- net N$10: now also C30.+; no longer C13.1
- net N$14: now also C30.-; no longer C13.2
- net N$19: now also C31.+; no longer C15.1
- net N$24: now also C31.-; no longer C15.2
- net N$26: now also C4.+; no longer C16.1
- net N$27: now also C32.-; no longer C17.2
- net N$6: now also D4.A, J4.PWR; no longer Q4.1, U2.X1
- net N$8: now also D1.A; no longer D2.+
- net N$9: now also D6.A; no longer D3.+
- net OUT+: now also C11.1, C20.1, C26.+, C5.1, U1.EN, U1.VIN, U2.EN, U2.VIN, U3.VIN; no longer C18.1, D1.K, R10.2, R6.1, R9.1, U$3.3V3, U$3.3V3.2, U2.VCC, U3.VCC, U4.VIN
- net R2IN: now also J5.4; no longer J2.3
- net RX: now also D6.C; no longer D3.-
- net T2OUT: now also J5.5; no longer J2.2
- net TX: now also D1.C; no longer D2.-
- net VCC: now also C25.+; no longer C4.1
Other:
- note added: "GPS"
- moved on the sheet: C12, D4, D5, D9, J4, JP2, JP3, X1-1, X1-2

Commit message: revisi jeck DC
Parts:
- removed J4: POWER_JACKSLT, SparkFun-Connectors:POWER_JACKSLT
- added J2: DCJ0202, con-jack:DCJ0202
Connections:
- net GND: now also J2.2, J2.3; no longer J4.GND, J4.GNDBREAK
- net N$6: now also J2.1; no longer J4.PWR
Changed lines of the file:
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@@
 <part name="C14" library="rcl" library_urn="urn:adsk.eagle:library:334" deviceset="C-EU" device="C0805K" package3d_urn="urn:adsk.eagle:package:23681/2" value="100nF"/>
 <part name="C10" library="rcl" library_urn="urn:adsk.eagle:library:334" deviceset="C-EU" device="C0805K" package3d_urn="urn:adsk.eagle:package:23681/2" value="100nF"/>
-<part name="J4" library="SparkFun-Connectors" library_urn="urn:adsk.eagle:library:513" deviceset="POWER_JACK" device="SLT" package3d_urn="urn:adsk.eagle:package:38222/1"/>
 <part name="U5" library="MAX232CSE" deviceset="MAX232CSE" device=""/>
 <part name="P+4" library="supply1" library_urn="urn:adsk.eagle:library:371" deviceset="VCC" device=""/>
@@
 <part name="D1" library="SML-LXT0805IW-TR" deviceset="SML-LXT0805IW-TR" device=""/>
 <part name="D6" library="SML-LXT0805IW-TR" deviceset="SML-LXT0805IW-TR" device=""/>
+<part name="J2" library="con-jack" library_urn="urn:adsk.eagle:library:154" deviceset="DCJ0202" device="" package3d_urn="urn:adsk.eagle:package:7491/1"/>
 </parts>
 <sheets>
@@
 <attribute name="VALUE" x="2.921" y="11.176" size="1.778" layer="96" rot="R270"/>
 </instance>
-<instance part="J4" gate="G$1" x="82.55" y="154.94" smashed="yes">
-<attribute name="VALUE" x="72.39" y="165.1" size="1.778" layer="96" font="vector"/>
-<attribute name="NAME" x="72.39" y="154.94" size="1.778" layer="95" font="vector"/>
-</instance>
 <instance part="U5" gate="A" x="106.68" y="-60.96" smashed="yes">
 <attribute name="NAME" x="93.98" y="-39.64" size="2.0828" layer="95" ratio="10" rot="SR0"/>
@@
 <attribute name="NAME" x="-62.49026875" y="-57.91513125" size="1.780740625" layer="95" rot="R90"/>
 <attribute name="VALUE" x="-54.60685" y="-57.91368125" size="1.77946875" layer="96" rot="R90"/>
+</instance>
+<instance part="J2" gate="G$1" x="77.47" y="160.02" smashed="yes">
+<attribute name="NAME" x="74.93" y="163.83" size="1.778" layer="95"/>
+<attribute name="VALUE" x="74.93" y="153.67" size="1.778" layer="96"/>
 </instance>
 </instances>
@@
 </segment>
 <segment>
-<pinref part="J4" gate="G$1" pin="GNDBREAK"/>
-<pinref part="J4" gate="G$1" pin="GND"/>
-<wire x1="85.09" y1="160.02" x2="85.09" y2="157.48" width="0.1524" layer="91"/>
 <wire x1="88.38" y1="144.56" x2="88.38" y2="139.7" width="0.1524" layer="91"/>
 <pinref part="C12" gate="G$1" pin="2"/>
@@
 <wire x1="88.38" y1="139.7" x2="109.22" y2="139.7" width="0.1524" layer="91"/>
 <wire x1="109.22" y1="139.7" x2="109.22" y2="137.16" width="0.1524" layer="91"/>
-<wire x1="85.09" y1="157.48" x2="85.09" y2="139.7" width="0.1524" layer="91"/>
-<junction x="85.09" y="157.48"/>
 <pinref part="GND8" gate="1" pin="GND"/>
 <wire x1="85.09" y1="139.7" x2="85.09" y2="137.16" width="0.1524" layer="91"/>
-<junction x="85.09" y="139.7"/>
 <pinref part="C26" gate="G$1" pin="-"/>
 <junction x="91.44" y="149.86"/>
+<pinref part="J2" gate="G$1" pin="3"/>
+<wire x1="85.09" y1="139.7" x2="85.09" y2="157.48" width="0.1524" layer="91"/>
+<junction x="85.09" y="139.7"/>
+<pinref part="J2" gate="G$1" pin="2"/>
+<wire x1="85.09" y1="160.02" x2="85.09" y2="157.48" width="0.1524" layer="91"/>
+<junction x="85.09" y="157.48"/>
 </segment>
 <segment>
@@
 <segment>
 <pinref part="D4" gate="G$1" pin="A"/>
-<pinref part="J4" gate="G$1" pin="PWR"/>
 <wire x1="93.98" y1="162.56" x2="85.09" y2="162.56" width="0.1524" layer="91"/>
-</segment>
-</net>
+<pinref part="J2" gate="G$1" pin="1"/>
+</segment>
+</net>
