File: monKWH+GPS/untitled.brd (EAGLE design)
At the start: 91 x 91 mm, 61 parts, among them J1 U.FL-R-SMT(01), J3 2172034-1, J4 POWER_JACKSLT, Q1 MMBT3904, Q2 MMBT3904, Q3 12MHz, Q4 MC-306, U2 DS1307Z+, U3 MAX3444EASA, U4 AMS1117, U5 MAX232CSE, X1 MSTBA2

Commit message: revisi rangkaian
Parts:
- removed C13, C15, C16, C17, C18: 10uf/50V, EEEFK1H100V:CAP_EEEFK1H100V
- removed D2: Tx, LHN974_RED_LED_1206:LEDC3216X120N
- removed D3: Rx, LHN974_RED_LED_1206:LEDC3216X120N
- removed G1: CR2032H, battery_cr2032:CR2032H
- removed J2: (no value), SparkFun-Connectors:DB9
- removed Q4: MC-306, crystal:MC-306
- removed R10, R6, R9: 10K, adafruit:M0805
- removed U$1: STEPDOWN_SY8205, STEPDOWN_SY8205:STEPDOWN_SY8205
- added C19, C20, C21, C5, C9: 10uF, rcl:C0805K
- added C25: 10uF/16v, rcl:153CLV-0505
- added C26, C28, C30, C31, C32: 10uF/16V, rcl:153CLV-0505
- added C27: 0.1uF/16V, rcl:153CLV-0505
- added C29: 0.1uf/16V, rcl:153CLV-0505
- added J5: RJ45-8N-B, RJ45-8N-B:TE_RJ45-8N-B
- added U1: RT9193-33GB, RT9193-33GB:SOT94P279X129-5N
- C11: value 10uf/50V -> 10uF; device EEEFK1H100V:CAP_EEEFK1H100V -> rcl:C0805K
- C4: value 10uf/50V -> 10uF/16V; device EEEFK1H100V:CAP_EEEFK1H100V -> rcl:153CLV-0505
- D1, D6: value 1N5819HW-7 -> SML-LXT0805IW-TR; device 1N5819HW-7:SOD3715X145N -> SML-LXT0805IW-TR:LEDC2012X120N
- U2: value DS1307Z+ -> RT9193-33GB; device DS1307Z_:SOIC127P600X175-8N -> RT9193-33GB:SOT94P279X129-5N
- U3: value MAX3444EASA -> RT9193-33GB; device MAX3444EASA:SOIC127P600X175-8N -> RT9193-33GB:SOT94P279X129-5N
- U4: value AMS1117 -> L80-R; device AMS1117:SOT229P700X180-4N -> L80-R:XCVR_L80-R
- moved POWER 106.3 mm to (75.6, 76.8), turned to 0 degrees
- moved R3 100.6 mm to (75.7, 73.2), turned to 180 degrees
- moved PROSES 95.1 mm to (75.9, 67.6), turned to 0 degrees
- moved R12 92.7 mm to (75.7, 71.0), turned to 180 degrees
- moved U2 87.7 mm to (27.0, 86.0), flipped to the bottom, turned to 180 degrees
- moved WARNING 86.6 mm to (75.9, 58.6), turned to 0 degrees
- moved U5 83.6 mm to (66.0, 79.0), turned to 270 degrees
- moved R13 83.6 mm to (75.5, 62.9), turned to 180 degrees
- moved C4 76.6 mm to (74.7, 49.7), turned to 0 degrees
- moved U3 73.4 mm to (34.2, 86.0), flipped to the bottom, turned to 180 degrees
- moved C12 71.7 mm to (30.8, 91.0), flipped to the bottom, turned to 0 degrees
- moved D4 67.9 mm to (40.8, 66.8), flipped to the bottom, turned to 0 degrees
- moved D6 64.3 mm to (59.4, 49.1), turned to 0 degrees
- moved D1 62.1 mm to (59.4, 51.4)
- moved D5 56.5 mm to (40.9, 64.0), flipped to the bottom, turned to 0 degrees
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Connections:
- removed net CLK: MD1.20
- removed net CMD: MD1.19
- removed net IO34: MD1.6
- removed net IO35: MD1.7
- removed net N$11: D4.A, U$1.OUT_VCC
- removed net N$15: G1.+, U2.3
- removed net N$18: R10.1, U2.7
- removed net N$20: D1.A, J2.9
- removed net N$23: D6.A, J4.PWR
- removed net N$7: Q4.4, U2.2
- removed net NC: MD1.32
- removed net RST_LAN: MD1.33, U$3.RST
- removed net SCL: R9.2, U2.6, U3.6
- removed net SD0: MD1.21
- removed net SD1: MD1.22
- removed net SD2: MD1.17
- removed net SD3: MD1.18
- removed net SDA: R6.2, U2.5, U3.5
- removed net SENSOR_VN: MD1.5
- removed net SENSOR_VP: MD1.4
- removed net VCC_DB9: D6.C, U$1.IN_VCC
- new net 3V3-LAN-GPS: C21.1, C27.+, C28.+, C29.+, U$3.3V3, U$3.3V3.2, U3.5, U4.4, U4.5
- new net 3V3-LORA-RS232: C19.1, C4.-, C7.2, C8.2, LORA-NICERF-V1.VCC, U2.5, U5.16
- new net EN-3V3-LAN-GPS: MD1.9, U3.3
- new net GPS_RXD: MD1.36, U4.1
- new net GPS_TXD: MD1.33, U4.2
- net 3V3: now also C9.1, U1.5; no longer C11.1, C16.2, C7.2, C8.2, LORA-NICERF-V1.VCC, U4.2, U4.4, U5.16
- net GND: now also C19.2, C20.2, C21.2, C25.-, C26.-, C27.-, C28.-, C29.-, C32.+, C5.2, C9.2, J5.10, J5.6, J5.9, U1.2, U2.2, U4.12, U4.3; no longer C17.1, C18.2, C4.2, G1.-, J2.5, U$1.IN_GND, U$1.OUT_GND, U2.4, U3.1, U3.3, U3.4, U3.7, U4.1
- net INT_LAN: no longer MD1.36
- net N$10: now also C30.+; no longer C13.1
- net N$14: now also C30.-; no longer C13.2
- net N$19: now also C31.+; no longer C15.1
- net N$24: now also C31.-; no longer C15.2
- net N$26: now also C4.+; no longer C16.1
- net N$27: now also C32.-; no longer C17.2
- net N$6: now also D4.A, J4.PWR; no longer Q4.1, U2.1
- net N$8: now also D1.A; no longer D2.+
- net N$9: now also D6.A; no longer D3.+
- net OUT+: now also C11.1, C20.1, C26.+, C5.1, U1.1, U1.3, U2.1, U2.3, U3.1; no longer C18.1, D1.C, R10.2, R6.1, R9.1, U$3.3V3, U$3.3V3.2, U2.8, U3.8, U4.3
- net R2IN: now also J5.4; no longer J2.3
- net RX: now also D6.C; no longer D3.-
- net T2OUT: now also J5.5; no longer J2.2
- net TX: now also D1.C; no longer D2.-
- net VCC: now also C25.+; no longer C4.1
Routing:
- net OUT+: track 332.3 -> 131.0 mm
- net 3V3: track 239.6 -> 87.0 mm, vias 6 -> 4
- net GND: track 644.1 -> 491.8 mm, vias 9 -> 134
- net 3V3-LORA-RS232: track 0.00 -> 148.3 mm, vias 0 -> 5
- net N$27: track 146.1 -> 9.35 mm
- net N$26: track 33.3 -> 141.1 mm
- net 3V3-LAN-GPS: track 0.00 -> 92.7 mm, vias 0 -> 4
- net VCC: track 238.6 -> 150.7 mm, vias 2 -> 5
- net EN-3V3-LAN-GPS: track 0.00 -> 85.8 mm, vias 0 -> 1
- net EN: track 103.3 -> 42.1 mm, vias 2 -> 1
- net INT_LAN: track 58.4 -> 0.00 mm
- net LED_PROSES: track 62.0 -> 4.18 mm
- net RX: track 71.4 -> 22.2 mm, vias 2 -> 1
- net RTS: track 74.6 -> 27.5 mm
- net N$19: track 75.5 -> 29.8 mm
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- added copper zone on layer 1, net GND
- added copper zone on layer 16, net GND
Other:
- board size 91 x 91 mm -> 66 x 60 mm

Commit message: revisi jeck DC
Parts:
- removed J4: POWER_JACKSLT, SparkFun-Connectors:POWER_JACK_SLOT
- added J2: DCJ0202, con-jack:DCJ0202
Connections:
- net GND: now also J2.2, J2.3; no longer J4.GND@1, J4.GND@2
- net N$6: now also J2.1; no longer J4.PWR
Routing:
- net ANT: track 18.9 -> 19.9 mm
- net N$6: track 53.5 -> 52.6 mm
- net GND: track 491.8 -> 491.0 mm
Changed lines of the file:
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@@
 <attribute name="PURCHASE-URL" value="https://pricing.snapeda.com/search/part/2172034-1/?ref=eda" x="14.254715625" y="-19.200728125" size="1.778" layer="27" rot="R270" display="off"/>
-</element>
-<element name="J4" library="SparkFun-Connectors" library_urn="urn:adsk.eagle:library:513" package="POWER_JACK_SLOT" package3d_urn="urn:adsk.eagle:package:38222/1" value="POWER_JACKSLT" x="14.62258125" y="36.88785" smashed="yes">
-<attribute name="NAME" x="18.12778125" y="39.04685" size="0.6096" layer="25" font="vector" ratio="20"/>
-<attribute name="PROD_ID" value="PRT-00119" x="93.36258125" y="6.40785" size="1.778" layer="27" display="off"/>
 </element>
 <element name="J5" library="RJ45-8N-B" package="TE_RJ45-8N-B" value="RJ45-8N-B" x="52.841059375" y="94.192640625" smashed="yes" rot="R180">
@@
 <attribute name="PRICE" value="None" x="59.4160625" y="49.135265625" size="1.778" layer="27" display="off"/>
 <attribute name="PURCHASE-URL" value="https://pricing.snapeda.com/search/part/SML-LXT0805IW-TR/?ref=eda" x="59.4160625" y="49.135265625" size="1.778" layer="27" display="off"/>
+</element>
+<element name="J2" library="con-jack" library_urn="urn:adsk.eagle:library:154" package="DCJ0202" package3d_urn="urn:adsk.eagle:package:7491/1" value="DCJ0202" x="18.9" y="47.3" smashed="yes">
+<attribute name="MF" value="" x="18.9" y="47.3" size="1.778" layer="27" display="off"/>
+<attribute name="MPN" value="" x="18.9" y="47.3" size="1.778" layer="27" display="off"/>
+<attribute name="NAME" x="15.09" y="52.38" size="1.27" layer="25"/>
+<attribute name="OC_FARNELL" value="unknown" x="18.9" y="47.3" size="1.778" layer="27" display="off"/>
+<attribute name="OC_NEWARK" value="unknown" x="18.9" y="47.3" size="1.778" layer="27" display="off"/>
+<attribute name="POPULARITY" value="17" x="18.9" y="47.3" size="1.778" layer="27" display="off"/>
+<attribute name="VALUE" x="13.82" y="37.14" size="1.27" layer="27" rot="R90"/>
 </element>
 </elements>
@@
 <contactref element="J5" pad="10"/>
 <contactref element="J5" pad="6"/>
-<contactref element="J4" pad="GND@1"/>
-<contactref element="J4" pad="GND@2"/>
 <contactref element="C12" pad="2"/>
 <contactref element="JP2" pad="2"/>
@@
 <contactref element="C29" pad="-"/>
 <contactref element="C32" pad="+"/>
-<wire x1="22.20258125" y1="47.68785" x2="22.20258125" y2="45.8547375" width="1.016" layer="16"/>
-<wire x1="22.20258125" y1="45.8547375" x2="20.668528125" y2="44.320684375" width="1.016" layer="16"/>
-<wire x1="20.668528125" y1="44.320684375" x2="17.269746875" y2="44.320684375" width="1.016" layer="16"/>
-<wire x1="17.269746875" y1="44.320684375" x2="17.20258125" y2="44.38785" width="1.016" layer="16"/>
 <wire x1="63.49371875" y1="42.233465625" x2="64.611184375" y2="41.116" width="0.2" layer="16"/>
 <wire x1="72.4829875" y1="41.116" x2="73.667765625" y2="42.300778125" width="0.2" layer="16"/>
@@
 <wire x1="18.773721875" y1="58.47225625" x2="18.773721875" y2="57.585671875" width="0.4064" layer="16"/>
 <wire x1="18.773721875" y1="57.585671875" x2="20.1416125" y2="56.21778125" width="0.4064" layer="16"/>
-<wire x1="20.1416125" y1="56.21778125" x2="20.25156875" y2="56.21778125" width="0.4064" layer="16"/>
-<wire x1="20.25156875" y1="56.21778125" x2="23.005165625" y2="56.21778125" width="0.4064" layer="16"/>
+<wire x1="20.1416125" y1="56.21778125" x2="23.005165625" y2="56.21778125" width="0.4064" layer="16"/>
 <wire x1="23.005165625" y1="56.21778125" x2="22.99625" y2="56.208865625" width="0.4064" layer="16"/>
 <wire x1="22.99625" y1="56.208865625" x2="22.97536875" y2="56.208865625" width="0.4064" layer="16"/>
 <via x="22.97536875" y="56.208865625" extent="1-16" drill="0.35"/>
-<wire x1="22.20258125" y1="47.68785" x2="20.25156875" y2="49.6388625" width="0.4064" layer="16"/>
-<wire x1="20.25156875" y1="49.6388625" x2="20.25156875" y2="56.21778125" width="0.4064" layer="16"/>
 <wire x1="67.640459375" y1="74.501346875" x2="67.640459375" y2="76.28745" width="0.4064" layer="1"/>
 <wire x1="67.640459375" y1="76.28745" x2="65.552815625" y2="78.37509375" width="0.4064" layer="1"/>
@@
 <via x="78.36264375" y="44.965734375" extent="1-16" drill="0.35"/>
 <via x="76.9802875" y="41.73833125" extent="1-16" drill="0.35"/>
+<contactref element="J2" pad="3"/>
+<contactref element="J2" pad="2"/>
+<wire x1="23.7" y1="47.3" x2="23.7" y2="45.9" width="1.016" layer="16"/>
+<wire x1="23.7" y1="45.9" x2="22.1" y2="44.3" width="1.016" layer="16"/>
+<wire x1="22.1" y1="44.3" x2="18.9" y2="44.3" width="1.016" layer="16"/>
+<wire x1="23.7" y1="47.3" x2="23.7" y2="55.505115625" width="0.4064" layer="16"/>
+<wire x1="23.7" y1="55.505115625" x2="22.99625" y2="56.208865625" width="0.4064" layer="16"/>
 </signal>
 <signal name="USB_P">
@@
 <contactref element="J1" pad="3"/>
 <wire x1="36.513721875" y1="58.06225625" x2="36.513721875" y2="56.806275" width="0.4064" layer="16"/>
-<via x="23.992303125" y="51.18056875" extent="1-16" drill="0.35"/>
-<wire x1="23.992303125" y1="51.18056875" x2="23.909971875" y2="51.2629" width="0.4064" layer="1"/>
-<wire x1="23.909971875" y1="51.2629" x2="23.909971875" y2="52.6507125" width="0.4064" layer="1"/>
-<wire x1="23.992303125" y1="51.18056875" x2="23.992303125" y2="53.436690625" width="0.4064" layer="16"/>
-<wire x1="23.992303125" y1="53.436690625" x2="26.3682625" y2="55.81265" width="0.4064" layer="16"/>
+<via x="25.592303125" y="50.98056875" extent="1-16" drill="0.35"/>
+<wire x1="25.592303125" y1="50.98056875" x2="24.692303125" y2="50.98056875" width="0.4064" layer="1"/>
+<wire x1="23.909971875" y1="52.6507125" x2="23.909971875" y2="51.7629" width="0.4064" layer="1"/>
+<wire x1="24.692303125" y1="50.98056875" x2="23.909971875" y2="51.7629" width="0.4064" layer="1"/>
+<wire x1="25.592303125" y1="50.98056875" x2="25.592303125" y2="55.036690625" width="0.4064" layer="16"/>
+<wire x1="25.592303125" y1="55.036690625" x2="26.3682625" y2="55.81265" width="0.4064" layer="16"/>
 <wire x1="26.3682625" y1="55.81265" x2="35.520096875" y2="55.81265" width="0.4064" layer="16"/>
 <wire x1="35.520096875" y1="55.81265" x2="36.513721875" y2="56.806275" width="0.4064" layer="16"/>
@@
 <signal name="N$6">
 <contactref element="D4" pad="A"/>
-<contactref element="J4" pad="PWR"/>
-<wire x1="17.20258125" y1="50.68785" x2="19.478534375" y2="52.963803125" width="0.2" layer="16"/>
-<wire x1="19.478534375" y1="52.963803125" x2="19.478534375" y2="55.52138125" width="0.2" layer="16"/>
-<wire x1="19.478534375" y1="55.52138125" x2="15.416246875" y2="59.58366875" width="0.2" layer="16"/>
+<wire x1="18.69995625" y1="56.299959375" x2="15.416246875" y2="59.58366875" width="0.2" layer="16"/>
 <wire x1="15.416246875" y1="71.585809375" x2="17.9653625" y2="74.134925" width="0.2" layer="16"/>
 <wire x1="17.9653625" y1="74.134925" x2="29.43183125" y2="74.134925" width="0.2" layer="16"/>
@@
 <wire x1="37.9980375" y1="66.77945" x2="37.99288125" y2="66.78460625" width="0.2" layer="16"/>
 <wire x1="15.416246875" y1="59.58366875" x2="15.416246875" y2="71.585809375" width="0.2" layer="16"/>
+<contactref element="J2" pad="1"/>
+<wire x1="18.9" y1="50.4" x2="18.9" y2="56.099915625" width="0.2" layer="16"/>
+<wire x1="18.9" y1="56.099915625" x2="18.69995625" y2="56.299959375" width="0.2" layer="16"/>
 </signal>
 <signal name="3V3-LORA-RS232">

Commit message: rangkaian Versi2
Routing:
- net IO0: track 75.2 -> 77.2 mm
- net ANT: track 19.9 -> 18.2 mm
- net N$6: track 52.6 -> 51.0 mm
- net DTR: track 23.0 -> 23.6 mm
- net GND: track 491.0 -> 490.8 mm, vias 134 -> 136
