File: monKWH+GPS v2/untitled.brd (EAGLE design)
At the start: 66 x 60 mm, 62 parts, among them J1 U.FL-R-SMT(01), J2 DCJ0202, J3 2172034-1, J5 RJ45-8N-B, Q1 MMBT3904, Q2 MMBT3904, Q3 12MHz, U1 RT9193-33GB, U2 RT9193-33GB, U3 RT9193-33GB, U4 L80-R, U5 MAX232CSE, X1 MSTBA2

Commit message: rangkaian Versi2
Parts:
- removed JP2: (no value), pinhead:1X02
- removed JP3: (no value), pinhead:1X03
- added PS1: PBO-5C-5, PBO-5C-5:CONV_PBO-5C-5
- moved J1 10.2 mm to (34.1, 55.1)
- moved R13 1.00 mm to (75.5, 63.9)
- moved WARNING 1.00 mm to (75.9, 59.6)
Connections:
- removed net N$17: D9.A, JP2.1
- new net N$15: PS1.2, X1.2
- net GND: now also PS1.5_1, PS1.5_2; no longer JP2.2
- net N$13: now also PS1.1; no longer JP3.1
- net N$16: now also D9.A, PS1.6; no longer JP3.3, X1.2
Routing:
- net N$16: track 5.75 -> 39.9 mm
- net N$15: track 0.00 -> 33.9 mm
- net N$17: track 26.4 -> 0.00 mm
- net N$13: track 5.75 -> 27.6 mm
- net GND: track 490.8 -> 508.0 mm, vias 136 -> 98
- net ANT: track 18.2 -> 10.1 mm
- net OUT+: track 131.0 -> 126.5 mm
- net N$6: track 51.0 -> 48.6 mm
- net N$26: track 141.1 -> 140.4 mm
- net IO0: track 77.2 -> 76.6 mm
- net MOSI_VSPI: vias 1 -> 5
Other:
- board size 66 x 60 mm -> 77 x 60 mm
