File: monKWH+GPS v2/untitled.sch (EAGLE design)
At the start: 62 parts, among them J1 U.FL-R-SMT(01), J3 2172034-1, J4 POWER_JACKSLT, J5 RJ45-8N-B, Q1 MMBT3904, Q2 MMBT3904, Q3 12MHz, U1 RT9193-33GB, U2 RT9193-33GB, U3 RT9193-33GB, U4 L80-R, U5 MAX232CSE, X1 MSTBA2

Commit message: rangkaian Versi2
Parts:
- removed J4: POWER_JACKSLT, SparkFun-Connectors:POWER_JACKSLT
- removed JP2: (no value), pinhead:PINHD-1X2
- removed JP3: (no value), pinhead:PINHD-1X3
- added J2: DCJ0202, con-jack:DCJ0202
- added PS1: PBO-5C-5, PBO-5C-5:PBO-5C-5
Connections:
- removed net N$17: D9.A, JP2.1
- removed net RST_LAN: U$3.RST
- new net N$15: PS1.AC(N), X1-2.1
- net GND: now also J2.2, J2.3, PS1.-VO; no longer J4.GND, J4.GNDBREAK, JP2.2
- net N$13: now also PS1.AC(L); no longer JP3.1
- net N$16: now also D9.A, PS1.+VO; no longer JP3.3, X1-2.1
- net N$6: now also J2.1; no longer J4.PWR
Other:
- moved on the sheet: D5, D9, X1-1, X1-2
