File: monKWH+GPS v2(HALIM)/untitled.brd (EAGLE design)
At the start: 88 x 60 mm, 71 parts, among them J3 10103594, J5 RJ45-8N-B, K1 G3MB202PDC12, K2 G3MB202PDC12, K4 G3MB202PDC12, Q1 MMBT3904, Q2 MMBT3904, Q3 12MHz, Q4 SS8550, Q5 SS8550, Q6 SS8550, U2 AMS1117, U5 MAX232CSE, X1 MSTBA2, X5 MSTBA3

Commit message: pengajuan komponen monkhw-HALIM
Connections:
- net MISO_VSPI: now also MD1.31; no longer MD1.37
- net MOSI_VSPI: now also MD1.37; no longer MD1.31
Routing:
- net MISO_VSPI: track 13.0 -> 20.3 mm
- net MOSI_VSPI: track 40.4 -> 33.2 mm
- net IO0: track 72.8 -> 73.6 mm
- net OUT+: track 232.5 -> 231.9 mm
