File: monKWH+GPS v2(HALIM)/untitled.sch (EAGLE design)
At the start: 71 parts, among them J3 10103594, J5 RJ45-8N-B, K1 G3MB202PDC12, K2 G3MB202PDC12, K4 G3MB202PDC12, Q1 MMBT3904, Q2 MMBT3904, Q3 12MHz, Q4 SS8550, Q5 SS8550, Q6 SS8550, U2 AMS1117, U5 MAX232CSE, X1 MSTBA2, X5 MSTBA3

Commit message: pengajuan komponen monkhw-HALIM
Connections:
- net MISO_VSPI: now also MD1.IO19; no longer MD1.IO23
- net MOSI_VSPI: now also MD1.IO23; no longer MD1.IO19
Changed lines of the file:
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@@
 </segment>
 <segment>
-<label x="-101.6" y="20.32" size="0.8128" layer="95" rot="R180" xref="yes"/>
-<wire x1="-101.6" y1="20.32" x2="-99.06" y2="20.32" width="0.1524" layer="91"/>
-<pinref part="MD1" gate="G$0" pin="IO19"/>
+<label x="-101.6" y="12.7" size="0.8128" layer="95" rot="R180" xref="yes"/>
+<wire x1="-101.6" y1="12.7" x2="-99.06" y2="12.7" width="0.1524" layer="91"/>
+<pinref part="MD1" gate="G$0" pin="IO23"/>
 </segment>
 </net>
@@
 </segment>
 <segment>
-<label x="-101.6" y="12.7" size="0.8128" layer="95" rot="R180" xref="yes"/>
-<wire x1="-101.6" y1="12.7" x2="-99.06" y2="12.7" width="0.1524" layer="91"/>
-<pinref part="MD1" gate="G$0" pin="IO23"/>
+<label x="-101.6" y="20.32" size="0.8128" layer="95" rot="R180" xref="yes"/>
+<wire x1="-101.6" y1="20.32" x2="-99.06" y2="20.32" width="0.1524" layer="91"/>
+<pinref part="MD1" gate="G$0" pin="IO19"/>
 </segment>
 </net>
